File: untitled.kicad_sch (KiCad schematic)
At the start: 19 parts, among them J4 motor

Commit message: controller fw added, unfinished
Parts:
- J4: value motor -> motor_L
Connections:
- net INH_B_L is gone; now on net INH: R16.2
- net INH_C_L is gone; now on net INH: R14.2
- net INH_A_L renamed INH
Changed lines of the file:
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@@
 		)
 	)
-	(global_label "INH_C_L"
+	(global_label "INH"
 		(shape input)
 		(at 91.44 119.38 180)
@@
 		)
 		(property "Intersheetrefs" "${INTERSHEET_REFS}"
-			(at 80.9557 119.38 0)
+			(at 85.189 119.38 0)
 			(effects
 				(font
@@
 		)
 	)
-	(global_label "INH_A_L"
+	(global_label "INH"
 		(shape input)
 		(at 101.6 57.15 180)
@@
 		)
 		(property "Intersheetrefs" "${INTERSHEET_REFS}"
-			(at 91.2971 57.15 0)
+			(at 95.349 57.15 0)
 			(effects
 				(font
@@
 		)
 	)
-	(global_label "INH_B_L"
+	(global_label "INH"
 		(shape input)
 		(at 93.98 88.9 180)
@@
 		)
 		(property "Intersheetrefs" "${INTERSHEET_REFS}"
-			(at 83.4957 88.9 0)
+			(at 87.729 88.9 0)
 			(effects
 				(font
@@
 			)
 		)
-		(property "Value" "motor"
+		(property "Value" "motor_L"
 			(at 196.85 85.09 0)
 			(effects

Commit message: still unfinished
Other:
- moved on the sheet: J4
Changed lines of the file:
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@@
+	(wire
+		(pts
+			(xy 149.86 83.82) (xy 205.74 83.82)
+		)
+		(stroke
+			(width 0)
+			(type default)
+		)
+	)
 	(wire
 		(pts
@@
 	(wire
 		(pts
-			(xy 152.4 86.36) (xy 190.5 86.36)
-		)
-		(stroke
-			(width 0)
-			(type default)
-		)
-	)
-	(wire
-		(pts
 			(xy 110.49 127) (xy 110.49 124.46)
 		)
@@
 	(wire
 		(pts
-			(xy 149.86 83.82) (xy 190.5 83.82)
-		)
-		(stroke
-			(width 0)
-			(type default)
-		)
-	)
-	(wire
-		(pts
 			(xy 148.59 116.84) (xy 152.4 116.84)
 		)
@@
 	(wire
 		(pts
-			(xy 152.4 81.28) (xy 190.5 81.28)
-		)
-		(stroke
-			(width 0)
-			(type default)
-		)
-	)
-	(wire
-		(pts
 			(xy 105.41 59.69) (xy 121.92 59.69)
 		)
@@
 	(wire
 		(pts
+			(xy 152.4 81.28) (xy 205.74 81.28)
+		)
+		(stroke
+			(width 0)
+			(type default)
+		)
+	)
+	(wire
+		(pts
 			(xy 120.65 114.3) (xy 121.92 114.3)
+		)
+		(stroke
+			(width 0)
+			(type default)
+		)
+	)
+	(wire
+		(pts
+			(xy 152.4 86.36) (xy 205.74 86.36)
 		)
 		(stroke
@@
 	(symbol
 		(lib_id "Connector:Conn_01x03_Socket")
-		(at 195.58 83.82 0)
+		(at 210.82 83.82 0)
 		(unit 1)
 		(exclude_from_sim no)
@@
 		(on_board yes)
 		(dnp no)
-		(fields_autoplaced yes)
 		(property "Reference" "J4"
-			(at 196.85 82.55 0)
+			(at 212.09 82.55 0)
 			(effects
 				(font
@@
 		)
 		(property "Value" "motor_L"
-			(at 196.85 85.09 0)
+			(at 212.09 85.09 0)
 			(effects
 				(font
@@
 		)
 		(property "Footprint" "TerminalBlock:TerminalBlock_MaiXu_MX126-5.0-03P_1x03_P5.00mm"
-			(at 195.58 83.82 0)
+			(at 210.82 83.82 0)
 			(effects
 				(font
@@
 		)
 		(property "Datasheet" "~"
-			(at 195.58 83.82 0)
+			(at 210.82 83.82 0)
 			(effects
 				(font
@@
 		)
 		(property "Description" ""
-			(at 195.58 83.82 0)
-			(effects
-				(font
+			(at 210.82 83.82 0)
+			(effects
+				(font
